Commit message: Added meshes and urdf's to complete SmartPick demo setup.

File: ssm_demo/urdf/itr_smartpick_description.urdf.xacro (robot description, xacro)
@@ -3,5 +3,7 @@
        name="itr_smartpick_description" >
 	<xacro:include filename="$(find denso_robot_descriptions)/vs087_description/urdf/vs087_macro.urdf.xacro" />
-	<xacro:include filename="$(find itr_smartpick_descriptions)/urdf/table.urdf.xacro" />
+	<xacro:include filename="$(find ssm_demo)/urdf/table.urdf.xacro" />
+	<xacro:include filename="$(find ssm_demo)/urdf/eyeT_support.urdf.xacro" />
+	<xacro:include filename="$(find ssm_demo)/urdf/bin.urdf.xacro" />
   	<!-- setup empty world -->
 	<link name="world"/>
@@ -14,3 +16,11 @@
   		<origin xyz="${table_width/2} ${table_length/2} ${table_height}" rpy="0 0 0"/>
 	</xacro:vs087>
+	<!-- include fake bin -->
+	<xacro:bin prefix="" parent="platform_base">
+  		<origin xyz="0.35 0.2 0" rpy="0 0 -${pi/2}"/>
+	</xacro:bin>
+	<!-- include eye-T + support-->
+	<xacro:eyeT_support prefix="" parent="world">
+  		<origin xyz="0 0 0" rpy="0 0 0"/>
+	</xacro:eyeT_support>
 </robot>

Commit message: Changed world frame to robot base_link to make IK intuitive.

File: ssm_demo/urdf/itr_smartpick_description.urdf.xacro (robot description, xacro)
@@ -10,9 +10,9 @@
 	<!-- include platform -->
 	<xacro:table prefix="" parent="world">
-  		<origin xyz="0 0 0" rpy="0 0 0"/>
+		<origin xyz="${-table_width/2} ${-table_length/2} ${-table_height}" rpy="0 0 0"/>
 	</xacro:table>
 	<!-- include robot -->
 	<xacro:vs087 prefix="" parent="world">
-  		<origin xyz="${table_width/2} ${table_length/2} ${table_height}" rpy="0 0 0"/>
+  		<origin xyz="0 0 0" rpy="0 0 0"/>
 	</xacro:vs087>
 	<!-- include fake bin -->
@@ -21,5 +21,5 @@
 	</xacro:bin>
 	<!-- include eye-T + support-->
-	<xacro:eyeT_support prefix="" parent="world">
+	<xacro:eyeT_support prefix="" parent="platform">
   		<origin xyz="0 0 0" rpy="0 0 0"/>
 	</xacro:eyeT_support>

Commit message: Added magnetic gripper to the robot description

File: ssm_demo/urdf/itr_smartpick_description.urdf.xacro (robot description, xacro)
@@ -6,4 +6,5 @@
 	<xacro:include filename="$(find ssm_demo)/urdf/eyeT_support.urdf.xacro" />
 	<xacro:include filename="$(find ssm_demo)/urdf/bin.urdf.xacro" />
+	<xacro:include filename="$(find ssm_demo)/urdf/suction_gripper_ipa_magnet.urdf.xacro" />
   	<!-- setup empty world -->
 	<link name="world"/>
@@ -24,3 +25,13 @@
   		<origin xyz="0 0 0" rpy="0 0 0"/>
 	</xacro:eyeT_support>
+    <!-- denso_flange_joint: Because real robot flange frame is rotated by PI/2 -->
+    <joint name="denso_flange_joint" type="fixed" >
+      <origin xyz="0 0 0" rpy="0 -${pi/2} 0" />
+      <parent link="ee_link" />
+      <child link="denso_flange" />
+    </joint>
+    <!--denso_flange: Because real robot flange frame is rotated by PI/2 -->
+    <link name="denso_flange"/>
+    <!-- tool -->
+    <xacro:suction_gripper_ipa prefix="" parent="denso_flange"/>
 </robot>
